Commit message: Add ultrasonic sensor integration with frame ID support
- Introduced a new link and joint for the ultrasonic sensor in the URDF file.
- Updated the Ultrasonic class constructor to accept a frame ID parameter.
- Modified the sensor initialization in the TurtleBot3 node to include the frame ID.
- Ensured the frame ID is set in the published messages for better sensor data context.

File: src/turtlebot3/turtlebot3_description/urdf/turtlebot3_burger.urdf (robot description, URDF)
Before this commit: robot turtlebot3_burger, 7 links, 6 joints
Links:
- added link ultrasonic_scan_link
Joints:
- added joint ultrasonic_scan_joint: type fixed, parent base_link, child ultrasonic_scan_link, origin xyz=0.12 0.0 0.08 rpy=0 0 0

Commit message: works enough

File: src/turtlebot3/turtlebot3_description/urdf/turtlebot3_burger.urdf (robot description, URDF)
Before this commit: robot turtlebot3_burger, 8 links, 7 joints
Joints:
- joint ultrasonic_scan_joint: origin xyz=0.12 0.0 0.08 rpy=0 0 0 -> xyz=-0.032 0 0.01 rpy=0 0 0

Commit message: update urdf to use namespace

File: src/turtlebot3/turtlebot3_description/urdf/turtlebot3_burger.urdf (robot description, URDF)
Before this commit: robot turtlebot3_burger, 8 links, 7 joints
Links:
- removed link ultrasonic_scan_link
- added link ${namespace}ultrasonic_scan_link
Joints:
- removed joint ultrasonic_scan_joint
- added joint ${namespace}ultrasonic_scan_joint: type fixed, parent ${namespace}base_link, child ${namespace}ultrasonic_scan_link, origin xyz=-0.032 0 0.01 rpy=0 0 0

Commit message: almost working

File: src/turtlebot3/turtlebot3_description/urdf/turtlebot3_burger.urdf (robot description, URDF)
Before this commit: robot turtlebot3_burger, 8 links, 7 joints
Links:
- added link ${namespace}gps_link
Joints:
- added joint ${namespace}gps_joint: type fixed, parent ${namespace}base_link, child ${namespace}gps_link, origin xyz=-0.032 0 0.068 rpy=0 0 0
